File: kicad/AntennaSwitchControl/AntennaSwitchControl.kicad_sch (KiCad schematic)
At the start: 120 parts, among them J1 Conn_01x12_Socket, J2 Conn_01x12_Socket, J3 POWER, K1 AHQSH112LM100G, K10 AHQSH112LM100G, K11 AHQSH112LM100G, K12 AHQSH112LM100G, K13 AHQSH112LM100G, K14 AHQSH112LM100G, K15 AHQSH112LM100G, K16 AHQSH112LM100G, K2 AHQSH112LM100G, K3 AHQSH112LM100G, K4 AHQSH112LM100G, K5 AHQSH112LM100G, K6 AHQSH112LM100G, K7 AHQSH112LM100G, K8 AHQSH112LM100G, K9 AHQSH112LM100G, Q1 2N7000, Q10 2N7000, Q11 2N7000, Q12 2N7000, Q13 2N7000, Q14 2N7000, Q15 2N7000, Q16 2N7000, Q2 2N7000, Q3 2N7000, Q4 2N7000, Q5 2N7000, Q6 2N7000, Q7 2N7000, Q8 2N7000, Q9 2N7000, SW1 Mode Button, U1 PicoW, U3 L7805

Commit message: add BOM, clean up schematic
Parts:
- R10: value 10 -> 100
- renumbered U3 to U2
Changed lines of the file:
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@@
 	(title_block
 		(title "AntennaSwitchControl")
+		(date "2024-10-30")
+		(rev "0.0.2")
 	)
 	(junction
@@
 			)
 		)
-		(property "Value" "10"
+		(property "Value" "100"
 			(at 238.76 57.15 90)
 			(effects
@@
 		(on_board yes)
 		(dnp no)
-		(property "Reference" "U3"
+		(property "Reference" "U2"
 			(at 82.55 216.1032 0)
 			(effects
@@
 			(project "16-relays"
 				(path "/10f319ac-f26a-460b-a674-c7bb32b891ee"
-					(reference "U3")
+					(reference "U2")
 					(unit 1)
 				)

Commit message: # Conflicts: #	src/switch_control/http_server.py
Parts:
- J1, J2: value Conn_01x12_Socket -> Terminal Block 12 terminal; footprint 705530116 -> Library:CUI_TBP04R1-500-12BE; Height 7.12 -> (none); Manufacturer_Name Molex -> Same Sky; Manufacturer_Part_Number 70553-0116 -> TBP04R1-500-12BE; Mouser Part Number 538-70553-0116 -> 179-TBP04R1-500-12BE; Mouser Price/Stock https://www.mouser.com/Search/Refine.aspx?Keyword=538-70553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 -> https://www.mouser.com/ProductDetail/179-TBP04R1-500-12BE
- J3: footprint 705530001 -> Library:CUI_TBP04R1-500-02BE; Height 7.12 -> (none); Manufacturer_Name Molex -> Same Sky; Manufacturer_Part_Number 70553-0001 -> TBP04R1-500-02BE; Mouser Part Number 538-70553-0001 -> 179-TBP04R1-500-02BE; Mouser Price/Stock https://www.mouser.co.uk/ProductDetail/Molex/70553-0001?qs=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 -> https://www.mouser.com/ProductDetail/179-TBP04R1-500-02BE; Part 26-60-4020 -> TBP04R1-500-02BE
- U1: footprint parts:RPi_PicoW_SMD_TH -> Library:RPi_PicoW_SMD_TH; symbol RPi_Pico:PicoW -> picow:Pico-W
Connections:
- net A1: now also U1.20 (GPIO15); no longer U1.17 (GPIO13)
- net A2: now also U1.19 (GPIO14); no longer U1.16 (GPIO12)
- net A3: now also U1.17 (GPIO13); no longer U1.15 (GPIO11)
- net A4: now also U1.16 (GPIO12); no longer U1.14 (GPIO10)
- net A5: now also U1.15 (GPIO11); no longer U1.12 (GPIO9)
- net A6: now also U1.14 (GPIO10); no longer U1.11 (GPIO8)
- net A7: now also U1.12 (GPIO9); no longer U1.10 (GPIO7)
- net A8: now also U1.11 (GPIO8); no longer U1.9 (GPIO6)
- net B1: now also U1.10 (GPIO7); no longer U1.32 (GPIO27_ADC1)
- net B2: now also U1.9 (GPIO6); no longer U1.31 (GPIO26_ADC0)
- net B3: now also U1.7 (GPIO5); no longer U1.27 (GPIO21)
- net B4: now also U1.6 (GPIO4); no longer U1.26 (GPIO20)
- net B5: now also U1.5 (GPIO3); no longer U1.25 (GPIO19)
- net B6: now also U1.4 (GPIO2); no longer U1.24 (GPIO18)
- net B7: now also U1.2 (GPIO1); no longer U1.22 (GPIO17)
- net B8: now also U1.1 (GPIO0); no longer U1.21 (GPIO16)
- net BLINKY: now also U1.22 (GPIO17); no longer U1.1 (GPIO0)
- net MODE: now reaches SW1.2
- net MODE: now also U1.21 (GPIO16); no longer U1.2 (GPIO1)
- net +3.3V: no longer names the net of U1.36 (3V3)
- no-connect marks 15 -> 16
Other:
- moved on the sheet: SW1
